File: hardware/interface-ascii-atmega2560/interface-ascii-2560.kicad_pcb (KiCad board)
At the start: 2 copper layers, 88.9 x 132.1 mm, 50 parts, among them J1 Apple 2, J10 Keyboard, J2 Apple 1, J3 UART, J4 Conn_01x05, J5 SOL-20, J6 Program, J7 Custom Connector 1 / Proto, J8 Conn_01x25, SW1 Options, U1 ATmega2560-16AU, Y1 16.000 MHz

Commit message: Add wiring for apple-II two-piece encoder replacement
Parts:
- J6: value Program -> Conn_01x16
- J8: value Conn_01x25 -> Apple II+ matrix
- moved J8 61.0 mm to (170.8, 168.6), turned to 180 degrees
Connections:
- J8 pad 10: Net-(J8-Pad10) -> /Row5
- J8 pad 11: Net-(J8-Pad11) -> /Col3
- J8 pad 12: Net-(J8-Pad12) -> /Row6
- J8 pad 13: Net-(J8-Pad13) -> /Col2
- J8 pad 14: Net-(J8-Pad14) -> /Col1
- J8 pad 15: Net-(J8-Pad15) -> /Row7
- J8 pad 16: Net-(J8-Pad16) -> /Row9
- J8 pad 17: Net-(J8-Pad17) -> /Col0
- J8 pad 18: Net-(J8-Pad18) -> /Row10
- J8 pad 19: Net-(J8-Pad19) -> /Col3
- J8 pad 2: Net-(J8-Pad2) -> /Col4
- J8 pad 20: Net-(J8-Pad20) -> /Row11
- J8 pad 21: Net-(J8-Pad21) -> /Col2
- J8 pad 22: Net-(J8-Pad22) -> /Row11
- J8 pad 23: Net-(J8-Pad23) -> /Row11
- J8 pad 24: Net-(J8-Pad24) -> /Col1
- J8 pad 3: Net-(J8-Pad3) -> /Col0
- J8 pad 4: Net-(J8-Pad4) -> /LED1
- J8 pad 5: Net-(J8-Pad5) -> /Row0
- J8 pad 6: Net-(J8-Pad6) -> /Row1
- J8 pad 7: Net-(J8-Pad7) -> /Row2
- J8 pad 8: Net-(J8-Pad8) -> /Row3
- J8 pad 9: Net-(J8-Pad9) -> /Row4
Routing:
- net /Row11: track 10.7 -> 159.6 mm, vias 0 -> 4
- net /Row10: track 16.7 -> 121.0 mm, vias 0 -> 3
- net /Row9: track 20.1 -> 123.3 mm, vias 0 -> 3
- net /Col0: track 103.4 -> 171.7 mm, vias 1 -> 6
- net /Row6: track 6.83 -> 66.8 mm, vias 0 -> 2
- net /Row3: track 6.73 -> 66.1 mm, vias 0 -> 1
- net /Col1: track 80.5 -> 139.7 mm, vias 2 -> 5
- net /Row2: track 6.74 -> 65.7 mm, vias 0 -> 1
- net /Row7: track 57.6 -> 115.7 mm, vias 0 -> 5
- net /Row4: track 6.72 -> 64.5 mm, vias 0 -> 1
- net /Col4: track 110.6 -> 167.3 mm, vias 3 -> 7
- net /Row5: track 6.83 -> 63.2 mm, vias 0 -> 1
- net /Col3: track 101.3 -> 152.9 mm, vias 3 -> 6
- net /Col2: track 91.4 -> 141.4 mm, vias 2 -> 4
- net /Row1: track 35.9 -> 65.8 mm, vias 0 -> 1
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